File: pcb/Dual6x09.sch (EAGLE design)
At the start: 7 parts, among them IC1 6x09, IC2 6x09

Commit message: Added DAT/MMU functionality support
Parts:
- added C1, C2: (no value), rcl:C-US025-025X050
- added IC3, IC4: 74LS245N, 74xx-us-jlb:74LS245N
- HD1, IC1, IC2: device micro-motorola:6809ER -> micro-motorola:MC6809ER
Connections:
- removed net N$1: CPU1-2.1, IC2A.TSC, R2.1
- removed net N$2: CPU1-2.3, IC1A.TSC, R1.1
- new net !CPU_1: CPU1-2.3, IC1A.TSC, IC3A.G, R1.1
- new net !CPU_2: CPU1-2.1, IC2A.TSC, IC4A.G, R2.1
- new net AVMA_1: IC1A.AVMA, IC3A.B3
- new net AVMA_2: IC2A.AVMA, IC4A.B3
- new net BA_1: IC1A.BA, IC3A.B4
- new net BA_2: IC2A.BA, IC4A.B4
- new net BS_1: IC1A.BS, IC3A.B2
- new net BS_2: IC2A.BS, IC4A.B2
- new net BUSY_1: IC1A.BUSY, IC3A.B5
- new net BUSY_2: IC2A.BUSY, IC4A.B5
- new net LIC_1: IC1A.LIC, IC3A.B1
- new net LIC_2: IC2A.LIC, IC4A.B1
- net AVMA: now also IC3A.A3, IC4A.A3
- net BA: now also IC3A.A4, IC4A.A4
- net BS: now also IC3A.A2, IC4A.A2
- net BUSY: now also IC3A.A5, IC4A.A5
- net GND: now also C1.2, C2.2, IC3A.B6, IC3A.B7, IC3A.B8, IC3A.DIR, IC3P.GND, IC4A.B6, IC4A.B7, IC4A.B8, IC4A.DIR, IC4P.GND
- net LIC: now also IC3A.A1, IC4A.A1
- net VCC: now also C1.1, C2.1, IC3P.VCC, IC4P.VCC
Other:
- moved on the sheet: CPU1-2, HD1, IC1, IC2, R1, R2
